File: Hardware/PCB/Ingenuity.kicad_pcb (KiCad board)
At the start: 4 copper layers, 65 x 30 mm, 45 parts, among them J1 Conn_ST_STDC14, J2 Conn_02x20_Odd_Even, J3 Conn_02x05_Odd_Even, J4 Conn_01x02, J5 Conn_01x02, J7 Conn_01x03, J8 Conn_01x03, J9 Conn_01x02, Q1 NMOS, Q2 NMOS, SW1 SW_SPDT, SW101 SW_Push, U1 STM32L412KBTx, U3 LSM6DSM, U4 AMS1117-3.3

Commit message: finalize pcb
Parts:
- moved D5 5.94 mm to (192.9, 48.2), turned to -90 degrees
- moved R6 5.09 mm to (192.9, 50.7), turned to 90 degrees
- moved D3 3.52 mm to (190.3, 48.2), turned to -90 degrees
- moved R4 3.21 mm to (190.3, 50.7)
- moved R2 3.06 mm to (187.7, 50.7)
- moved D1 2.72 mm to (187.7, 48.2), turned to -90 degrees
- moved J8 0.91 mm to (198.0, 65.0)
- moved C3 0.38 mm to (192.9, 63.6)
- renumbered C9 to C1, C5 to C2, C6 to C3, C1 to C4, C7 to C5, C8 to C6, C3 to C7, C11 to C8, C2 to C9, D103 to D1, D1 to D2, D101 to D3, D2 to D4, D102 to D5, D3 to D6, J4 to J1, J3 to J2, J2 to J3, J7 to J4, J8 to J5, J9 to J6, J5 to J7, J1 to J8, Q2 to Q1, Q1 to Q2, R2 to R1, R3 to R10, R103 to R2, R4 to R3, R101 to R4, R102 to R6, R6 to R7, R1 to R8, SW101 to SW2, U2 to U1, U1 to U2, U4 to U3, U3 to U4
Routing:
- net +3.3V: track 33.9 -> 21.7 mm, vias 8 -> 10
- net GND: track 17.9 -> 22.5 mm, vias 33 -> 39
- net LED3: track 1.04 -> 5.71 mm
- net LED2: track 1.51 -> 4.98 mm
- net LED1: track 1.59 -> 4.81 mm
- net USART1_TX: track 5.99 -> 4.86 mm
- net Net-(D1-A): track 2.30 -> 1.19 mm
- net USART1_RX: track 9.89 -> 8.94 mm, vias 2 -> 0
- net Net-(D3-A): track 2.11 -> 1.19 mm
- net NRST: track 30.8 -> 30.0 mm, vias 2 -> 3
- net PWM3: track 12.3 -> 11.7 mm
Other:
- board text added: "+ Batt -"
- board text added: "+3V3"
- board text added: "+5V"
- board text added: "1"
- board text added: "Mot1"
- board text added: "Mot2"
- board text added: "NRST"
- board text added: "Servo1"
- board text added: "Servo2"
- board text added: "Vbat"
